Commit message: mpc code modify

File: kwj_description/urdf/kwj.gazebo.xacro (robot description, xacro)
@@ -1,5 +1,5 @@
 <?xml version="1.0"?>
 <robot name="KWJBot" xmlns:xacro="http://ros.org/wiki/xacro">
-  <xacro:arg name="laser_visual"  default="true"/>
+  <xacro:arg name="laser_visual"  default="false"/>
   <xacro:arg name="camera_visual" default="false"/>
   <xacro:arg name="imu_visual"    default="true"/>

File: kwj_description/urdf/kwj.urdf.xacro (robot description, xacro)
@@ -35,5 +35,5 @@
     <parent link="base_link"/>
     <child link="camera_link"/>
-    <origin xyz="0.08 0 0.13" rpy="0 0 0"/>
+    <origin xyz="0.15 0 0.1" rpy="0 0 0"/>
   </joint>
   <link name="camera_link">
@@ -41,5 +41,5 @@
       <origin xyz="0 0 0" rpy="0 0 0"/>
       <geometry>
-        <box size="0.03 0.07 0.03"/>
+        <box size="0.03 0.085 0.025"/>
       </geometry>
       <material name="black"/>

Commit message: i modify description file

File: kwj_description/urdf/kwj.gazebo.xacro (robot description, xacro)
@@ -3,5 +3,5 @@
   <xacro:arg name="laser_visual"  default="false"/>
   <xacro:arg name="camera_visual" default="false"/>
-  <xacro:arg name="imu_visual"    default="true"/>
+  <xacro:arg name="imu_visual"    default="false"/>
   <gazebo reference="base_link">
     <material>Gazebo/DarkGrey</material>
@@ -11,5 +11,5 @@
     <mu2>0.1</mu2>
     <kp>500000.0</kp>
-    <kd>10.0</kd>
+    <kd>10</kd>
     <minDepth>0.001</minDepth>
     <maxVel>0.1</maxVel>
@@ -21,5 +21,5 @@
     <mu2>0.1</mu2>
     <kp>500000.0</kp>
-    <kd>10.0</kd>
+    <kd>10</kd>
     <minDepth>0.001</minDepth>
     <maxVel>0.1</maxVel>
@@ -30,8 +30,9 @@
     <mu1>0.1</mu1>
     <mu2>0.1</mu2>
-    <kp>1000000.0</kp>
-    <kd>100.0</kd>
+    <kp>500000.0</kp>
+    <kd>10</kd>
     <minDepth>0.001</minDepth>
     <maxVel>1.0</maxVel>
+    <fdir1>1 0 0</fdir1>
     <material>Gazebo/FlatBlack</material>
   </gazebo>
@@ -70,12 +71,12 @@
    </gazebo>
   <gazebo>
-    <plugin name="differential_drive_controller" filename="libgazebo_ros_diff_drive.so">
+    <plugin name="kwj_controller" filename="libgazebo_ros_diff_drive.so">
       <commandTopic>cmd_vel</commandTopic>
-      <odometryTopic>odometry/filtered</odometryTopic>
+      <odometryTopic>/odometry/filtered</odometryTopic>
       <odometryFrame>odom</odometryFrame>
       <odometrySource>world</odometrySource>
       <publishOdomTF>true</publishOdomTF>
       <robotBaseFrame>base_footprint</robotBaseFrame>
-      <publishWheelTF>true</publishWheelTF>
+      <publishWheelTF>false</publishWheelTF>
       <publishTf>true</publishTf>
       <publishWheelJointState>true</publishWheelJointState>
@@ -87,5 +88,5 @@
       <wheelDiameter>0.067</wheelDiameter>
       <wheelAcceleration>1</wheelAcceleration>
-      <wheelTorque>5</wheelTorque>
+      <wheelTorque>10</wheelTorque>
       <rosDebugLevel>na</rosDebugLevel>
     </plugin>

File: kwj_description/urdf/kwj.urdf.xacro (robot description, xacro)
@@ -3,166 +3,173 @@
     <xacro:include filename="$(find kwj_description)/urdf/kwj.gazebo.xacro"/>
     <link name="base_footprint"/>
+    <link name="base_link">
+      <inertial>
+        <origin xyz="0 0 0" rpy="0 0 0"/>
+        <mass value="0.35" />
+        <inertia ixx="0.00178" ixy="0" ixz="0"
+                 iyy="0.00178" iyz="0"
+                 izz="0.00178" />
+        </inertial>
+      <collision>
+        <origin xyz="0 0 0" rpy="0 0 0"/>
+        <geometry>
+          <box size="0.155 0.2 0.15"/>
+        </geometry>
+      </collision>
+      <visual>
+        <origin xyz="0 0 0" rpy="0 0 0"/>
+        <geometry>
+          <mesh filename="package://kwj_description/meshes/base_link.stl" scale="1.0 1.0 1.0"/>
+        </geometry>
+        <material name="grey">
+          <color rgba="0.5 0.5 0.5 1"/>
+        </material>
+      </visual>
+    </link>
     <joint name="base_joint" type="fixed">
-       <parent link="base_footprint"/>
-       <child link="base_link"/>
-       <origin xyz="0 0 0.065" rpy="0 0 0"/>
+         <parent link="base_footprint"/>
+         <child link="base_link"/>
+         <origin xyz="0 0 0.065" rpy="0 0 0"/>
+      </joint>
+    <joint name="camera_joint" type="fixed">
+      <parent link="base_link"/>
+      <child link="camera_link"/>
+      <origin xyz="0.15 0 0.05" rpy="0 0 0"/>
     </joint>
-  <link name="base_link">
-    <inertial>
-      <origin xyz="0 0 0" rpy="0 0 0"/>
-      <mass value="1.0" />
-      <inertia ixx="0.001" ixy="0" ixz="0"
-               iyy="0.001" iyz="0"
-               izz="0.001" />
+    <link name="camera_link">
+      <visual>
+        <origin xyz="0 0 0" rpy="0 0 0"/>
+        <geometry>
+         <box size="0.03 0.085 0.025"/>
+        </geometry>
+        <material name="black"/>
+      </visual>
+      <collision>
+        <origin xyz="0.015 0 -0.0065" rpy="0 0 0"/>
+        <geometry>
+          <box size="0.05 0.05 0.025"/>
+        </geometry>
+      </collision>
+      <inertial>
+        <mass value="0.072"/>
+        <origin xyz="0 0 0" rpy="0 0 0"/>
+        <inertia ixx="0.00005235" iyy="0.00005235" izz="0.00005235" ixy="0" ixz="0" iyz="0"/>
       </inertial>
-    <collision>
-      <origin xyz="0 0 0" rpy="0 0 0"/>
-      <geometry>
-        <box size="0.155 0.2 0.25"/>
-      </geometry>
-    </collision>
-    <visual>
-      <origin xyz="0 0 0" rpy="0 0 0"/>
-      <geometry>
-        <mesh filename="package://kwj_description/meshes/base_link.stl" scale="1.0 1.0 1.0"/>
-      </geometry>
-      <material name="grey">
-        <color rgba="0.5 0.5 0.5 1"/>
-      </material>
-    </visual>
-  </link>
-  <joint name="camera_joint" type="fixed">
-    <parent link="base_link"/>
-    <child link="camera_link"/>
-    <origin xyz="0.15 0 0.1" rpy="0 0 0"/>
-  </joint>
-  <link name="camera_link">
-    <visual>
-      <origin xyz="0 0 0" rpy="0 0 0"/>
-      <geometry>
-        <box size="0.03 0.085 0.025"/>
-      </geometry>
-      <material name="black"/>
-    </visual>
-    <collision>
-      <origin xyz="0 0 0" rpy="0 0 0"/>
-      <geometry>
-        <box size="0.1 0.1 0.05"/>
-      </geometry>
-    </collision>
-    <inertial>
-      <mass value="0.1"/>
-      <origin xyz="0 0 0" rpy="0 0 0"/>
-      <inertia ixx="0.01" iyy="0.01" izz="0.01" ixy="0" ixz="0" iyz="0"/>
-    </inertial>
-  </link>
-   <joint name="wheel_left_joint" type="fixed">
-    <parent link="base_link"/>
-    <child link="wheel_left_link"/>
-    <origin xyz="-0.0355 0.075 -0.02" rpy="-1.57 0 0"/>
-    <axis xyz="0 0 1"/>
-   </joint>
-   <link name="wheel_left_link">
-    <visual>
-      <origin xyz="0 0 0" rpy="0 0 0"/>
+    </link>
+     <joint name="wheel_left_joint" type="continuous">
+      <parent link="base_link"/>
+      <child link="wheel_left_link"/>
+      <origin xyz="-0.0355 0.106 -0.0515" rpy="-1.57 0 0"/>
+      <axis xyz="0 0 1"/>
+     </joint>
+     <link name="wheel_left_link">
+      <visual>
+        <origin xyz="0 0 0" rpy="0 0 1.57"/>
+          <geometry>
+           <cylinder length="0.026" radius="0.0335"/>
+          </geometry>
+        <material name="dark"/>
+      </visual>
+      <collision>
+        <origin xyz="0 0 0" rpy="0 0 0"/>
         <geometry>
-         <cylinder length="0.026" radius="0.0335"/>
+          <cylinder length="0.026" radius="0.0335"/>
         </geometry>
-      <material name="dark"/>
-    </visual>
-    <collision>
-      <origin xyz="0 0 0" rpy="0 0 0"/>
-      <geometry>
-        <cylinder length="0.026" radius="0.0335"/>
-      </geometry>
-    </collision>
-    <inertial>
-      <origin xyz="0 0 0" />
-      <mass value="2.8498940e-02" />
-      <inertia ixx="0.001" ixy="0" ixz="0"
-               iyy="0.001" iyz="0"
-               izz="0.001" />
+      </collision>
+      <inertial>
+        <origin xyz="0 0 0" />
+        <mass value="1.2" />
+        <inertia ixx="0.00020535" ixy="0" ixz="0"
+                 iyy="0.00020535" iyz="0"
+                 izz="0.00020535" />
+        </inertial>
+    </link>
+     <joint name="wheel_right_joint" type="continuous">
+      <parent link="base_link"/>
+      <child link="wheel_right_link"/>
+      <origin xyz="-0.0355 -0.106 -0.0515" rpy="-1.57 0 0"/>
+      <axis xyz="0 0 1"/>
+     </joint>
+     <link name="wheel_right_link">
+      <visual>
+        <origin xyz="0 0 0" rpy="0 0 1.57"/>
+         <geometry>
+           <cylinder length="0.026" radius="0.0335"/>
+         </geometry>
+        <material name="dark"/>
+      </visual>
+      <collision>
+        <origin xyz="0 0 0" rpy="0 0 0"/>
+        <geometry>
+          <cylinder length="0.026" radius="0.0335"/>
+        </geometry>
+      </collision>
+      <inertial>
+        <origin xyz="0 0 0" />
+        <mass value="1.2" />
+        <inertia ixx="0.00020535" ixy="0" ixz="0"
+                 iyy="0.00020535" iyz="0"
+                 izz="0.00020535" />
+        </inertial>
+    </link>
+    <joint name="caster_front_joint" type="fixed">
+      <parent link="base_link"/>
+      <child link="caster_front_link"/>
+      <origin xyz="0.1 0 -0.07" rpy="-1.57 0 0"/>
+    </joint>
+    <link name="caster_front_link">
+      <visual>
+        <origin xyz="0 0 0" rpy="0 0 0"/>
+         <geometry>
+           <cylinder length="0.015" radius="0.0175"/>
+         </geometry>
+        <material name="dark"/>
+      </visual>
+      <collision>
+        <origin xyz="0 0.001 0" rpy="0 0 0"/>
+        <geometry>
+          <cylinder length="0.016" radius="0.015"/>
+        </geometry>
+      </collision>
+      <inertial>
+        <origin xyz="0 0 0" />
+        <mass value="0.022" />
+        <inertia ixx="0.00000336875" ixy="0" ixz="0"
+                 iyy="0.00000336875" iyz="0"
+                 izz="0.00000336875" />
       </inertial>
-  </link>
-   <joint name="wheel_right_joint" type="fixed">
-    <parent link="base_link"/>
-    <child link="wheel_right_link"/>
-    <origin xyz="-0.0355 -0.0775 -0.02" rpy="-1.57 0 0"/>
-    <axis xyz="0 0 1"/>
-   </joint>
-   <link name="wheel_right_link">
-    <visual>
-      <origin xyz="0 0 0" rpy="0 0 0"/>
-       <geometry>
-         <cylinder length="0.026" radius="0.0335"/>
-       </geometry>
-      <material name="dark"/>
-    </visual>
-    <collision>
-      <origin xyz="0 0 0" rpy="0 0 0"/>
-      <geometry>
-        <cylinder length="0.026" radius="0.0335"/>
-      </geometry>
-    </collision>
-    <inertial>
-      <origin xyz="0 0 0" />
-      <mass value="2.8498940e-02" />
-      <inertia ixx="0.001" ixy="0" ixz="0"
-               iyy="0.001" iyz="0"
-               izz="0.001" />
+    </link>
+     <joint name="imu_joint" type="fixed">
+      <parent link="base_link"/>
+      <child link="imu_link"/>
+      <origin xyz="-0.07 0 0" rpy="0 0 0"/>
+     </joint>
+     <link name="imu_link"/>
+     <joint name="scan_joint" type="fixed">
+      <parent link="base_link"/>
+      <child link="laser_link"/>
+      <origin xyz="0.11 0 0.18" rpy="0 0 0"/>
+     </joint>
+     <link name="laser_link">
+      <visual>
+        <origin xyz="0 0 0" rpy="0 0 0"/>
+          <geometry>
+           <cylinder length="0.0105" radius="0.03435"/>
+        </geometry>
+        <material name="dark"/>
+      </visual>
+      <collision>
+        <origin xyz="-0.015 0 -0.0065" rpy="0 0 0"/>
+        <geometry>
+          <cylinder length="0.0105" radius="0.03435"/>
+        </geometry>
+      </collision>
+      <inertial>
+        <mass value="0.178" />
+        <origin xyz="0 0 0" />
+        <inertia ixx="0.0002225" ixy="0.0" ixz="0.0"
+                 iyy="0.0002225" iyz="0.0"
+                 izz="0.0002225" />
       </inertial>
-  </link>
-  <joint name="caster_front_joint" type="fixed">
-    <parent link="base_link"/>
-    <child link="caster_front_link"/>
-    <origin xyz="0.193 0.01 -0.02" rpy="0 0 -1.57"/>
-  </joint>
-  <link name="caster_front_link">
-    <collision>
-      <origin xyz="0 0 0" rpy="0 0 0"/>
-      <geometry>
-        <cylinder length="0.016" radius="0.0175"/>
-      </geometry>
-    </collision>
-    <inertial>
-      <origin xyz="0 0 0" />
-      <mass value="0.005" />
-      <inertia ixx="0.001" ixy="0.0" ixz="0.0"
-               iyy="0.001" iyz="0.0"
-               izz="0.001" />
-    </inertial>
-  </link>
-   <joint name="imu_joint" type="fixed">
-    <parent link="base_link"/>
-    <child link="imu_link"/>
-    <origin xyz="-0.07 0 0" rpy="0 0 0"/>
-   </joint>
-   <link name="imu_link"/>
-   <joint name="scan_joint" type="fixed">
-    <parent link="base_link"/>
-    <child link="laser_link"/>
-    <origin xyz="0.11 0 0.18" rpy="0 0 0"/>
-   </joint>
-   <link name="laser_link">
-    <visual>
-      <origin xyz="0 0 0" rpy="0 0 0"/>
-        <geometry>
-         <cylinder length="0.0105" radius="0.03435"/>
-      </geometry>
-      <material name="dark"/>
-    </visual>
-    <collision>
-      <origin xyz="0.055 0 0.2" rpy="0 0 0"/>
-      <geometry>
-        <cylinder length="0.0105" radius="0.03435"/>
-      </geometry>
-    </collision>
-    <inertial>
-      <mass value="0.114" />
-      <origin xyz="0 0 0" />
-      <inertia ixx="0.001" ixy="0.0" ixz="0.0"
-               iyy="0.001" iyz="0.0"
-               izz="0.001" />
-    </inertial>
-  </link>
+    </link>
 </robot>

Commit message: I make preparation gazebo simulation

File: kwj_description/urdf/kwj.gazebo.xacro (robot description, xacro)
@@ -21,5 +21,5 @@
     <mu2>0.1</mu2>
     <kp>500000.0</kp>
-    <kd>10</kd>
+    <kd>100</kd>
     <minDepth>0.001</minDepth>
     <maxVel>0.1</maxVel>
@@ -31,7 +31,7 @@
     <mu2>0.1</mu2>
     <kp>500000.0</kp>
-    <kd>10</kd>
+    <kd>100</kd>
     <minDepth>0.001</minDepth>
-    <maxVel>1.0</maxVel>
+    <maxVel>0.1</maxVel>
     <fdir1>1 0 0</fdir1>
     <material>Gazebo/FlatBlack</material>
@@ -62,5 +62,5 @@
       <plugin name="camera_controller" filename="libgazebo_ros_camera.so">
         <always_on>true</always_on>
-        <update_rate>30.0</update_rate>
+        <update_rate>5.0</update_rate>
         <cameraName>camera</cameraName>
         <imageTopicName>/camera/depth/image_rect_raw</imageTopicName>
@@ -72,11 +72,11 @@
   <gazebo>
     <plugin name="kwj_controller" filename="libgazebo_ros_diff_drive.so">
-      <commandTopic>cmd_vel</commandTopic>
+      <commandTopic>/cmd_vel</commandTopic>
       <odometryTopic>/odometry/filtered</odometryTopic>
       <odometryFrame>odom</odometryFrame>
       <odometrySource>world</odometrySource>
       <publishOdomTF>true</publishOdomTF>
-      <robotBaseFrame>base_footprint</robotBaseFrame>
-      <publishWheelTF>false</publishWheelTF>
+      <robotBaseFrame>base_link</robotBaseFrame>
+      <publishWheelTF>true</publishWheelTF>
       <publishTf>true</publishTf>
       <publishWheelJointState>true</publishWheelJointState>
@@ -100,5 +100,5 @@
       <serviceName>imu_service</serviceName>
       <gaussianNoise>0.0</gaussianNoise>
-      <updateRate>10</updateRate>
+      <updateRate>0</updateRate>
       <imu>
         <noise>
@@ -125,5 +125,5 @@
       <pose>0 0 0 0 0 0</pose>
       <visualize>$(arg laser_visual)</visualize>
-      <update_rate>10</update_rate>
+      <update_rate>5</update_rate>
       <ray>
         <scan>
@@ -138,5 +138,5 @@
           <min>0.1</min>
           <max>10</max>
-          <resolution>0.05</resolution>
+          <resolution>0.015</resolution>
         </range>
         <noise>

File: kwj_description/urdf/kwj.urdf.xacro (robot description, xacro)
@@ -5,9 +5,9 @@
     <link name="base_link">
       <inertial>
-        <origin xyz="0 0 0" rpy="0 0 0"/>
-        <mass value="0.35" />
-        <inertia ixx="0.00178" ixy="0" ixz="0"
-                 iyy="0.00178" iyz="0"
-                 izz="0.00178" />
+        <origin xyz="0 0 0.065" rpy="0 0 0"/>
+        <mass value="0.8343"/>
+        <inertia ixx="0.005259" ixy="0.005470" ixz="0.003567"
+                 iyy="0.005710" iyz="0.005603"
+                 izz="0.005524" />
         </inertial>
       <collision>
@@ -35,5 +35,5 @@
       <parent link="base_link"/>
       <child link="camera_link"/>
-      <origin xyz="0.15 0 0.05" rpy="0 0 0"/>
+      <origin xyz="0.15 0 0.115" rpy="0 0 0"/>
     </joint>
     <link name="camera_link">
@@ -41,7 +41,9 @@
         <origin xyz="0 0 0" rpy="0 0 0"/>
         <geometry>
-         <box size="0.03 0.085 0.025"/>
+          <mesh filename="package://kwj_description/meshes/camera_gazebo.stl" scale="1.0 1.0 1.0"/>
         </geometry>
-        <material name="black"/>
+        <material name="grey">
+          <color rgba="0.5 0.5 0.5 1"/>
+        </material>
       </visual>
       <collision>
@@ -52,7 +54,7 @@
       </collision>
       <inertial>
-        <mass value="0.072"/>
+        <mass value="3.07365e-05"/>
         <origin xyz="0 0 0" rpy="0 0 0"/>
-        <inertia ixx="0.00005235" iyy="0.00005235" izz="0.00005235" ixy="0" ixz="0" iyz="0"/>
+        <inertia ixx="3.073649974518707e-05" iyy="8.101563506798558e-06" izz="4.316406649983658e-05" ixy="0" ixz="0" iyz="0"/>
       </inertial>
     </link>
@@ -79,8 +81,8 @@
       <inertial>
         <origin xyz="0 0 0" />
-        <mass value="1.2" />
-        <inertia ixx="0.00020535" ixy="0" ixz="0"
-                 iyy="0.00020535" iyz="0"
-                 izz="0.00020535" />
+        <mass value="0.1004" />
+        <inertia ixx="3.3800152140578693e-05" ixy="0" ixz="0"
+                 iyy="5.628900326021782e-05" iyz="0"
+                 izz="3.380015380915577e-05" />
         </inertial>
     </link>
@@ -107,8 +109,8 @@
       <inertial>
         <origin xyz="0 0 0" />
-        <mass value="1.2" />
-        <inertia ixx="0.00020535" ixy="0" ixz="0"
-                 iyy="0.00020535" iyz="0"
-                 izz="0.00020535" />
+        <mass value="0.1004" />
+        <inertia ixx="3.3800152140578693e-05" ixy="0" ixz="0"
+                 iyy="5.628900326021782e-05" iyz="0"
+                 izz="3.380015380915577e-05" />
         </inertial>
     </link>
@@ -116,13 +118,15 @@
       <parent link="base_link"/>
       <child link="caster_front_link"/>
-      <origin xyz="0.1 0 -0.07" rpy="-1.57 0 0"/>
+      <origin xyz="0.14 0 -0.07" rpy="-1.57 0 0"/>
     </joint>
     <link name="caster_front_link">
       <visual>
-        <origin xyz="0 0 0" rpy="0 0 0"/>
-         <geometry>
-           <cylinder length="0.015" radius="0.0175"/>
-         </geometry>
-        <material name="dark"/>
+        <origin xyz="0 0 0" rpy="-1.57 0 -1.57"/>
+        <geometry>
+          <mesh filename="package://kwj_description/meshes/caster_gazebo.stl" scale="1.0 1.0 1.0"/>
+        </geometry>
+        <material name="grey">
+          <color rgba="0.5 0.5 0.5 1"/>
+        </material>
       </visual>
       <collision>
@@ -134,8 +138,8 @@
       <inertial>
         <origin xyz="0 0 0" />
-        <mass value="0.022" />
-        <inertia ixx="0.00000336875" ixy="0" ixz="0"
-                 iyy="0.00000336875" iyz="0"
-                 izz="0.00000336875" />
+        <mass value="0.01439" />
+        <inertia ixx="1.21919e-06" ixy="1.70883e-06" ixz="1.21919e-06"
+                 iyy="2.19848e-06" iyz="1.70883e-06"
+                 izz="1.21919e-06" />
       </inertial>
     </link>
@@ -154,8 +158,10 @@
       <visual>
         <origin xyz="0 0 0" rpy="0 0 0"/>
-          <geometry>
-           <cylinder length="0.0105" radius="0.03435"/>
+        <geometry>
+          <mesh filename="package://kwj_description/meshes/lidar_gazebo.stl" scale="1.0 1.0 1.0"/>
         </geometry>
-        <material name="dark"/>
+        <material name="grey">
+          <color rgba="0.5 0.5 0.5 1"/>
+        </material>
       </visual>
       <collision>
@@ -166,9 +172,9 @@
       </collision>
       <inertial>
-        <mass value="0.178" />
+        <mass value="0.04659" />
         <origin xyz="0 0 0" />
-        <inertia ixx="0.0002225" ixy="0.0" ixz="0.0"
-                 iyy="0.0002225" iyz="0.0"
-                 izz="0.0002225" />
+        <inertia ixx="1.41344e-05" ixy="0" ixz="0"
+                 iyy="1.40144e-05" iyz="0"
+                 izz="2.74129e-05" />
       </inertial>
     </link>
