Commit message: i add fuzzy-neuron control

File: kwj_description/urdf/kwj.gazebo.xacro (robot description, xacro)
@@ -3,5 +3,5 @@
   <xacro:arg name="laser_visual"  default="false"/>
   <xacro:arg name="camera_visual" default="false"/>
-  <xacro:arg name="imu_visual"    default="false"/>
+  <xacro:arg name="imu_visual"    default="true"/>
   <gazebo reference="base_link">
     <material>Gazebo/DarkGrey</material>
@@ -11,5 +11,5 @@
     <mu2>0.1</mu2>
     <kp>500000.0</kp>
-    <kd>10</kd>
+    <kd>10.0</kd>
     <minDepth>0.001</minDepth>
     <maxVel>0.1</maxVel>
@@ -21,5 +21,5 @@
     <mu2>0.1</mu2>
     <kp>500000.0</kp>
-    <kd>100</kd>
+    <kd>10.0</kd>
     <minDepth>0.001</minDepth>
     <maxVel>0.1</maxVel>
@@ -30,9 +30,8 @@
     <mu1>0.1</mu1>
     <mu2>0.1</mu2>
-    <kp>500000.0</kp>
-    <kd>100</kd>
+    <kp>1000000.0</kp>
+    <kd>100.0</kd>
     <minDepth>0.001</minDepth>
-    <maxVel>0.1</maxVel>
-    <fdir1>1 0 0</fdir1>
+    <maxVel>1.0</maxVel>
     <material>Gazebo/FlatBlack</material>
   </gazebo>
@@ -62,5 +61,5 @@
       <plugin name="camera_controller" filename="libgazebo_ros_camera.so">
         <always_on>true</always_on>
-        <update_rate>5.0</update_rate>
+        <update_rate>30.0</update_rate>
         <cameraName>camera</cameraName>
         <imageTopicName>/camera/depth/image_rect_raw</imageTopicName>
@@ -71,7 +70,7 @@
    </gazebo>
   <gazebo>
-    <plugin name="kwj_controller" filename="libgazebo_ros_diff_drive.so">
-      <commandTopic>/cmd_vel</commandTopic>
-      <odometryTopic>/odometry/filtered</odometryTopic>
+    <plugin name="differential_drive_controller" filename="libgazebo_ros_diff_drive.so">
+      <commandTopic>cmd_vel</commandTopic>
+      <odometryTopic>odometry/filtered</odometryTopic>
       <odometryFrame>odom</odometryFrame>
       <odometrySource>world</odometrySource>
@@ -88,5 +87,5 @@
       <wheelDiameter>0.067</wheelDiameter>
       <wheelAcceleration>1</wheelAcceleration>
-      <wheelTorque>10</wheelTorque>
+      <wheelTorque>5</wheelTorque>
       <rosDebugLevel>na</rosDebugLevel>
     </plugin>
@@ -100,5 +99,5 @@
       <serviceName>imu_service</serviceName>
       <gaussianNoise>0.0</gaussianNoise>
-      <updateRate>0</updateRate>
+      <updateRate>10</updateRate>
       <imu>
         <noise>
@@ -125,5 +124,5 @@
       <pose>0 0 0 0 0 0</pose>
       <visualize>$(arg laser_visual)</visualize>
-      <update_rate>5</update_rate>
+      <update_rate>10</update_rate>
       <ray>
         <scan>
@@ -138,5 +137,5 @@
           <min>0.1</min>
           <max>10</max>
-          <resolution>0.015</resolution>
+          <resolution>0.05</resolution>
         </range>
         <noise>

File: kwj_description/urdf/kwj.urdf.xacro (robot description, xacro)
@@ -59,5 +59,5 @@
       </inertial>
     </link>
-     <joint name="wheel_left_joint" type="continuous">
+     <joint name="wheel_left_joint" type="fixed">
       <parent link="base_link"/>
       <child link="wheel_left_link"/>
@@ -87,5 +87,5 @@
         </inertial>
     </link>
-     <joint name="wheel_right_joint" type="continuous">
+     <joint name="wheel_right_joint" type="fixed">
       <parent link="base_link"/>
       <child link="wheel_right_link"/>

Commit message: i add making-global-planning code in local planning code

File: kwj_description/urdf/kwj.gazebo.xacro (robot description, xacro)
@@ -72,14 +72,14 @@
     <plugin name="differential_drive_controller" filename="libgazebo_ros_diff_drive.so">
       <commandTopic>cmd_vel</commandTopic>
-      <odometryTopic>odometry/filtered</odometryTopic>
+      <odometryTopic>odom</odometryTopic>
       <odometryFrame>odom</odometryFrame>
       <odometrySource>world</odometrySource>
       <publishOdomTF>false</publishOdomTF>
       <robotBaseFrame>base_footprint</robotBaseFrame>
-      <publishWheelTF>false</publishWheelTF>
+      <publishWheelTF>true</publishWheelTF>
       <publishTf>true</publishTf>
       <publishWheelJointState>true</publishWheelJointState>
       <legacyMode>false</legacyMode>
-      <updateRate>50</updateRate>
+      <updateRate>15</updateRate>
       <leftJoint>wheel_left_joint</leftJoint>
       <rightJoint>wheel_right_joint</rightJoint>
@@ -99,5 +99,5 @@
       <serviceName>imu_service</serviceName>
       <gaussianNoise>0.0</gaussianNoise>
-      <updateRate>0</updateRate>
+      <updateRate>5</updateRate>
       <imu>
         <noise>
@@ -124,5 +124,5 @@
       <pose>0 0 0 0 0 0</pose>
       <visualize>$(arg laser_visual)</visualize>
-      <update_rate>5</update_rate>
+      <update_rate>10</update_rate>
       <ray>
         <scan>
@@ -130,6 +130,6 @@
             <samples>360</samples>
             <resolution>1</resolution>
-            <min_angle>-1.57</min_angle>
-            <max_angle>1.57</max_angle>
+            <min_angle>-180</min_angle>
+            <max_angle>180</max_angle>
           </horizontal>
         </scan>

File: kwj_description/urdf/kwj.urdf.xacro (robot description, xacro)
@@ -59,5 +59,5 @@
       </inertial>
     </link>
-     <joint name="wheel_left_joint" type="fixed">
+     <joint name="wheel_left_joint" type="continuous">
       <parent link="base_link"/>
       <child link="wheel_left_link"/>
@@ -87,5 +87,5 @@
         </inertial>
     </link>
-     <joint name="wheel_right_joint" type="fixed">
+     <joint name="wheel_right_joint" type="continuous">
       <parent link="base_link"/>
       <child link="wheel_right_link"/>

Commit message: i fixed dwa code

File: kwj_description/urdf/kwj.gazebo.xacro (robot description, xacro)
@@ -3,5 +3,5 @@
   <xacro:arg name="laser_visual"  default="false"/>
   <xacro:arg name="camera_visual" default="false"/>
-  <xacro:arg name="imu_visual"    default="true"/>
+  <xacro:arg name="imu_visual"    default="false"/>
   <gazebo reference="base_link">
     <material>Gazebo/DarkGrey</material>
@@ -61,5 +61,5 @@
       <plugin name="camera_controller" filename="libgazebo_ros_camera.so">
         <always_on>true</always_on>
-        <update_rate>10.0</update_rate>
+        <update_rate>0</update_rate>
         <cameraName>camera</cameraName>
         <imageTopicName>/camera/depth/image_rect_raw</imageTopicName>
@@ -74,5 +74,5 @@
       <odometryTopic>odom</odometryTopic>
       <odometryFrame>odom</odometryFrame>
-      <odometrySource>world</odometrySource>
+      <odometrySource>encoder</odometrySource>
       <publishOdomTF>false</publishOdomTF>
       <robotBaseFrame>base_footprint</robotBaseFrame>
@@ -81,11 +81,11 @@
       <publishWheelJointState>true</publishWheelJointState>
       <legacyMode>false</legacyMode>
-      <updateRate>15</updateRate>
+      <updateRate>5</updateRate>
       <leftJoint>wheel_left_joint</leftJoint>
       <rightJoint>wheel_right_joint</rightJoint>
       <wheelSeparation>0.212</wheelSeparation>
       <wheelDiameter>0.067</wheelDiameter>
-      <wheelAcceleration>3</wheelAcceleration>
-      <wheelTorque>3</wheelTorque>
+      <wheelAcceleration>1</wheelAcceleration>
+      <wheelTorque>2</wheelTorque>
       <rosDebugLevel>na</rosDebugLevel>
     </plugin>
@@ -99,5 +99,5 @@
       <serviceName>imu_service</serviceName>
       <gaussianNoise>0.0</gaussianNoise>
-      <updateRate>5</updateRate>
+      <updateRate>0</updateRate>
       <imu>
         <noise>
@@ -124,5 +124,5 @@
       <pose>0 0 0 0 0 0</pose>
       <visualize>$(arg laser_visual)</visualize>
-      <update_rate>10</update_rate>
+      <update_rate>0</update_rate>
       <ray>
         <scan>

File: kwj_description/urdf/kwj.urdf.xacro (robot description, xacro)
@@ -83,7 +83,7 @@
         <mass value="0.1004" />
         <inertia ixx="3.3800152140578693e-05" ixy="0" ixz="0"
-                 iyy="5.628900326021782e-05" iyz="0"
+                 iyy="5.628900326021782e-05"  iyz="0"
                  izz="3.380015380915577e-05" />
-        </inertial>
+       </inertial>
     </link>
      <joint name="wheel_right_joint" type="continuous">

Commit message: i made no problems in graph_slam and test with another model

File: kwj_description/urdf/kwj.gazebo.xacro (robot description, xacro)
@@ -8,28 +8,28 @@
   </gazebo>
   <gazebo reference="wheel_left_link">
-    <mu1>0.1</mu1>
-    <mu2>0.1</mu2>
-    <kp>50000000.0</kp>
-    <kd>100</kd>
+    <mu1>0.4</mu1>
+    <mu2>0.4</mu2>
+    <kp>5000.0</kp>
+    <kd>10</kd>
     <minDepth>0.001</minDepth>
     <maxVel>0.1</maxVel>
-    <fdir1>1 0 0</fdir1>
+    <fdir1>1 1 0</fdir1>
     <material>Gazebo/FlatBlack</material>
   </gazebo>
   <gazebo reference="wheel_right_link">
-    <mu1>0.1</mu1>
-    <mu2>0.1</mu2>
-    <kp>50000000.0</kp>
-    <kd>100</kd>
+    <mu1>0.4</mu1>
+    <mu2>0.4</mu2>
+    <kp>5000.0</kp>
+    <kd>10</kd>
     <minDepth>0.001</minDepth>
     <maxVel>0.1</maxVel>
-    <fdir1>1 0 0</fdir1>
+    <fdir1>1 1 0</fdir1>
     <material>Gazebo/FlatBlack</material>
   </gazebo>
   <gazebo reference="caster_front_link">
-    <mu1>0.1</mu1>
-    <mu2>0.1</mu2>
-    <kp>100000000.0</kp>
-    <kd>200</kd>
+    <mu1>0.4</mu1>
+    <mu2>0.4</mu2>
+    <kp>10000.0</kp>
+    <kd>20</kd>
     <minDepth>0.001</minDepth>
     <maxVel>1.0</maxVel>
@@ -74,12 +74,12 @@
       <odometryTopic>odom</odometryTopic>
       <odometryFrame>odom</odometryFrame>
-      <odometrySource>encoder</odometrySource>
-      <publishOdomTF>false</publishOdomTF>
-      <robotBaseFrame>base_link</robotBaseFrame>
-      <publishWheelTF>true</publishWheelTF>
+      <odometrySource>world</odometrySource>
+      <publishOdomTF>true</publishOdomTF>
+      <robotBaseFrame>base_footprint</robotBaseFrame>
+      <publishWheelTF>false</publishWheelTF>
       <publishTf>true</publishTf>
       <publishWheelJointState>true</publishWheelJointState>
       <legacyMode>false</legacyMode>
-      <updateRate>5</updateRate>
+      <updateRate>100</updateRate>
       <leftJoint>wheel_left_joint</leftJoint>
       <rightJoint>wheel_right_joint</rightJoint>
@@ -87,5 +87,5 @@
       <wheelDiameter>0.067</wheelDiameter>
       <wheelAcceleration>1</wheelAcceleration>
-      <wheelTorque>2</wheelTorque>
+      <wheelTorque>10</wheelTorque>
       <rosDebugLevel>na</rosDebugLevel>
     </plugin>
@@ -124,5 +124,5 @@
       <pose>0 0 0 0 0 0</pose>
       <visualize>$(arg laser_visual)</visualize>
-      <update_rate>0</update_rate>
+      <update_rate>5</update_rate>
       <ray>
         <scan>
@@ -137,5 +137,5 @@
           <min>0.1</min>
           <max>10</max>
-          <resolution>0.05</resolution>
+          <resolution>0.015</resolution>
         </range>
         <noise>

File: kwj_description/urdf/kwj.urdf.xacro (robot description, xacro)
@@ -5,5 +5,5 @@
     <link name="base_link">
       <inertial>
-        <origin xyz="0 0 0.065" rpy="0 0 0"/>
+        <origin xyz="0 0 0" rpy="0 0 0"/>
         <mass value="0.8343"/>
         <inertia ixx="0.005259" ixy="0.005470" ixz="0.003567"
@@ -18,5 +18,5 @@
       </collision>
       <visual>
-        <origin xyz="0 0 0" rpy="0 0 0"/>
+        <origin xyz="-0.025 0 -0.02" rpy="0 0 0"/>
         <geometry>
           <mesh filename="package://kwj_description/meshes/base_link.stl" scale="1.0 1.0 1.0"/>
@@ -62,5 +62,5 @@
       <parent link="base_link"/>
       <child link="wheel_left_link"/>
-      <origin xyz="-0.0355 0.106 -0.0515" rpy="-1.57 0 0"/>
+      <origin xyz="-0.0335 0.106 -0.0515" rpy="-1.57 0 0"/>
       <axis xyz="0 0 1"/>
      </joint>
@@ -90,5 +90,5 @@
       <parent link="base_link"/>
       <child link="wheel_right_link"/>
-      <origin xyz="-0.0355 -0.106 -0.0515" rpy="-1.57 0 0"/>
+      <origin xyz="-0.0335 -0.106 -0.0515" rpy="-1.57 0 0"/>
       <axis xyz="0 0 1"/>
      </joint>
@@ -122,5 +122,5 @@
     <link name="caster_front_link">
       <visual>
-        <origin xyz="0 0 0" rpy="-1.57 0 -1.57"/>
+        <origin xyz="0 0 0" rpy="1.57 0 1.57"/>
         <geometry>
           <mesh filename="package://kwj_description/meshes/caster_gazebo.stl" scale="1.0 1.0 1.0"/>
@@ -139,6 +139,6 @@
         <origin xyz="0 0 0" />
         <mass value="0.01439" />
-        <inertia ixx="1.21919e-06" ixy="1.70883e-06" ixz="1.21919e-06"
-                 iyy="2.19848e-06" iyz="1.70883e-06"
+        <inertia ixx="1.21919e-06" ixy="0" ixz="0"
+                 iyy="2.19848e-06" iyz="0"
                  izz="1.21919e-06" />
       </inertial>

Commit message: i modified model and made graph_slam map

File: kwj_description/urdf/kwj.gazebo.xacro (robot description, xacro)
@@ -8,28 +8,28 @@
   </gazebo>
   <gazebo reference="wheel_left_link">
-    <mu1>0.4</mu1>
-    <mu2>0.4</mu2>
-    <kp>5000.0</kp>
+    <mu1>10</mu1>
+    <mu2>10</mu2>
+    <kp>100000.0</kp>
     <kd>10</kd>
     <minDepth>0.001</minDepth>
-    <maxVel>0.1</maxVel>
-    <fdir1>1 1 0</fdir1>
+    <maxVel>1.0</maxVel>
+    <fdir1>1 0 0</fdir1>
     <material>Gazebo/FlatBlack</material>
   </gazebo>
   <gazebo reference="wheel_right_link">
-    <mu1>0.4</mu1>
-    <mu2>0.4</mu2>
-    <kp>5000.0</kp>
+    <mu1>10</mu1>
+    <mu2>10</mu2>
+    <kp>100000.0</kp>
     <kd>10</kd>
     <minDepth>0.001</minDepth>
-    <maxVel>0.1</maxVel>
-    <fdir1>1 1 0</fdir1>
+    <maxVel>1.0</maxVel>
+    <fdir1>1 0 0</fdir1>
     <material>Gazebo/FlatBlack</material>
   </gazebo>
   <gazebo reference="caster_front_link">
-    <mu1>0.4</mu1>
-    <mu2>0.4</mu2>
-    <kp>10000.0</kp>
-    <kd>20</kd>
+    <mu1>0.1</mu1>
+    <mu2>0.1</mu2>
+    <kp>1000000.0</kp>
+    <kd>100</kd>
     <minDepth>0.001</minDepth>
     <maxVel>1.0</maxVel>
@@ -39,4 +39,5 @@
     <sensor type="imu" name="imu">
       <always_on>true</always_on>
+      <update_rate>50</update_rate>
       <visualize>$(arg imu_visual)</visualize>
     </sensor>
@@ -81,5 +82,5 @@
       <publishWheelJointState>true</publishWheelJointState>
       <legacyMode>false</legacyMode>
-      <updateRate>100</updateRate>
+      <updateRate>10</updateRate>
       <leftJoint>wheel_left_joint</leftJoint>
       <rightJoint>wheel_right_joint</rightJoint>
@@ -87,6 +88,5 @@
       <wheelDiameter>0.067</wheelDiameter>
       <wheelAcceleration>1</wheelAcceleration>
-      <wheelTorque>10</wheelTorque>
-      <rosDebugLevel>na</rosDebugLevel>
+      <wheelTorque>100</wheelTorque>
     </plugin>
   </gazebo>
@@ -99,5 +99,5 @@
       <serviceName>imu_service</serviceName>
       <gaussianNoise>0.0</gaussianNoise>
-      <updateRate>0</updateRate>
+      <updateRate>100</updateRate>
       <imu>
         <noise>
@@ -105,7 +105,7 @@
           <rate>
             <mean>0.0</mean>
-            <stddev>2e-4</stddev>
-            <bias_mean>0.0000075</bias_mean>
-            <bias_stddev>0.0000008</bias_stddev>
+            <stddev>1.7e-2</stddev>
+            <bias_mean>0.1</bias_mean>
+            <bias_stddev>0.001</bias_stddev>
           </rate>
           <accel>
@@ -122,7 +122,7 @@
     <material>Gazebo/FlatBlack</material>
     <sensor type="ray" name="lds_lfcd_sensor">
-      <pose>0 0 0 0 0 0</pose>
+      <pose>0 0 0 0 0 1.57079631</pose>
       <visualize>$(arg laser_visual)</visualize>
-      <update_rate>5</update_rate>
+      <update_rate>1500</update_rate>
       <ray>
         <scan>
@@ -135,12 +135,12 @@
         </scan>
         <range>
-          <min>0.1</min>
+          <min>0.05</min>
           <max>10</max>
-          <resolution>0.015</resolution>
+          <resolution>0.009</resolution>
         </range>
         <noise>
           <type>gaussian</type>
           <mean>0.0</mean>
-          <stddev>0.001</stddev>
+          <stddev>0.01</stddev>
         </noise>
       </ray>

File: kwj_description/urdf/kwj.urdf.xacro (robot description, xacro)
@@ -82,6 +82,6 @@
         <origin xyz="0 0 0" />
         <mass value="0.1004" />
-        <inertia ixx="3.3800152140578693e-05" ixy="0" ixz="0"
-                 iyy="5.628900326021782e-05"  iyz="0"
+        <inertia ixx="3.3800152140578693e-05" ixy="4.91450e-11" ixz="3.68838e-11"
+                 iyy="5.628900326021782e-05"  iyz="4.91450e-11"
                  izz="3.380015380915577e-05" />
        </inertial>
@@ -110,6 +110,6 @@
         <origin xyz="0 0 0" />
         <mass value="0.1004" />
-        <inertia ixx="3.3800152140578693e-05" ixy="0" ixz="0"
-                 iyy="5.628900326021782e-05" iyz="0"
+        <inertia ixx="3.3800152140578693e-05" ixy="4.91450e-11" ixz="3.68838e-11"
+                 iyy="5.628900326021782e-05" iyz="4.91450e-11"
                  izz="3.380015380915577e-05" />
         </inertial>
@@ -118,5 +118,5 @@
       <parent link="base_link"/>
       <child link="caster_front_link"/>
-      <origin xyz="0.14 0 -0.07" rpy="-1.57 0 0"/>
+      <origin xyz="0.115 -0.005 -0.07" rpy="-1.57 0 0"/>
     </joint>
     <link name="caster_front_link">
@@ -153,5 +153,5 @@
       <parent link="base_link"/>
       <child link="laser_link"/>
-      <origin xyz="0.11 0 0.18" rpy="0 0 0"/>
+      <origin xyz="0.11 0 0.25" rpy="0 0 0"/>
      </joint>
      <link name="laser_link">

Commit message: modify model and detect_object

File: kwj_description/urdf/kwj.gazebo.xacro (robot description, xacro)
@@ -2,5 +2,5 @@
 <robot name="KWJBot" xmlns:xacro="http://ros.org/wiki/xacro">
   <xacro:arg name="laser_visual"  default="false"/>
-  <xacro:arg name="camera_visual" default="false"/>
+  <xacro:arg name="camera_visual" default="true"/>
   <xacro:arg name="imu_visual"    default="false"/>
   <gazebo reference="base_link">
@@ -44,8 +44,11 @@
     <material>Gazebo/Grey</material>
   </gazebo>
-  <gazebo>
-   <sensor type="camera" name="camera_sensor">
+   <gazebo reference="camera_link">
+   <material>Gazebo/Red</material>
+   <sensor type="camera" name="camera">
+      <pose>0 0 0 0 0 0</pose>
+      <visualize>$(arg camera_visual)</visualize>
       <always_on>true</always_on>
-      <update_rate>0</update_rate>
+      <update_rate>30</update_rate>
       <camera>
         <horizontal_fov>1.39626</horizontal_fov>
@@ -62,7 +65,9 @@
       <plugin name="camera_controller" filename="libgazebo_ros_camera.so">
         <always_on>true</always_on>
-        <update_rate>0</update_rate>
+        <update_rate>30</update_rate>
+        <min_depth>0.1</min_depth>
+        <max_depth>100.0</max_depth>
         <cameraName>camera</cameraName>
-        <imageTopicName>/camera/depth/image_rect_raw</imageTopicName>
+        <imageTopicName>/camera/color/image_raw</imageTopicName>
         <cameraInfoTopicName>camera/camera_info</cameraInfoTopicName>
         <frameName>camera_link</frameName>
