Commit message: update docker ros-robot

File: kwj_description/urdf/kwj.urdf.xacro (robot description, xacro)
@@ -41,5 +41,5 @@
       <origin xyz="0 0 0" rpy="0 0 0"/>
       <geometry>
-        <box size="0.1 0.1 0.05"/>
+        <box size="0.03 0.07 0.03"/>
       </geometry>
       <material name="black"/>

Commit message: modify model

File: kwj_description/urdf/kwj.urdf.xacro (robot description, xacro)
@@ -6,8 +6,8 @@
       <inertial>
         <origin xyz="0 0 0" rpy="0 0 0"/>
-        <mass value="0.8343"/>
-        <inertia ixx="0.005259" ixy="0.005470" ixz="0.003567"
-                 iyy="0.005710" iyz="0.005603"
-                 izz="0.005524" />
+        <mass value="0.01"/>
+        <inertia ixx="5.259e-03" ixy="5.470e-05" ixz="3.567e-04"
+                 iyy="5.710e-03" iyz="5.603e-06"
+                 izz="5.524e-02" />
         </inertial>
       <collision>
@@ -82,5 +82,5 @@
         <origin xyz="0 0 0" />
         <mass value="0.1004" />
-        <inertia ixx="3.3800152140578693e-05" ixy="4.91450e-11" ixz="3.68838e-11"
+        <inertia ixx="3.3800152140578693e-05" ixy="4.91450e-11" ixz="3.68838e-09"
                  iyy="5.628900326021782e-05"  iyz="4.91450e-11"
                  izz="3.380015380915577e-05" />
@@ -110,5 +110,5 @@
         <origin xyz="0 0 0" />
         <mass value="0.1004" />
-        <inertia ixx="3.3800152140578693e-05" ixy="4.91450e-11" ixz="3.68838e-11"
+        <inertia ixx="3.3800152140578693e-05" ixy="4.91450e-11" ixz="3.68838e-09"
                  iyy="5.628900326021782e-05" iyz="4.91450e-11"
                  izz="3.380015380915577e-05" />
